File: Hardware/KiCad/projects/rp2040_v0/rp2040_v0/reaction_control_wheel.kicad_sch (KiCad schematic)
At the start: 15 parts, among them J22 Conn_02x05_Odd_Even, J23 Screw_Terminal_01x02, U11 AMS1117-5.0, U12 DRV8837

Commit message: Remove reaction wheel LDO. Add jumper to select power source.
Parts:
- removed C35, C36: 10uF, Capacitor_SMD:C_0805_2012Metric, symbol Device:C_Small
- removed U11: AMS1117-5.0, Package_TO_SOT_SMD:SOT-223-3_TabPin2, symbol Regulator_Linear:AMS1117-5.0
- added J16: Conn_01x03, Connector_PinHeader_2.54mm:PinHeader_1x03_P2.54mm_Vertical, symbol Connector_Generic:Conn_01x03
Connections:
- net Protected_VBATT+: now also J16.1 (Pin_1)
- net 5v_MOTOR renamed MOTOR_POWER
- net MOTOR_POWER: now also J16.2 (Pin_2)
- new net +5V: J16.3 (Pin_3)
Other:
- note added: "Jumper selects which power source to run the motors from. Be aware of what else is on the 5v rail if using that. Make sure the LDO can handle it."
- note removed: "Likely only 250mA used but give it a full 1A just in case"
