File: Hardware/KiCad/projects/rp2040_v0/rp2040_v0/rp2040_v0.kicad_sch (KiCad schematic)
At the start: 52 parts, among them J1 Conn_01x03, J10 Conn_01x01, J11 Conn_01x02, J12 Screw_Terminal_01x02, J2 Conn_01x02, J3 Conn_01x03, J4 Conn_01x01, J5 USB_B_Micro, J6 Conn_01x01, J7 Conn_01x01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

Commit message: Update the flash chip footprint to use default kicad instead of generated one. The 3d model was messed up and I wanted assurance the footprint was not the issue.
Parts:
- U1: footprint easyeda2kicad:SOIC-8_L5.3-W5.3-P1.27-LS8.0-BL -> Package_SO:SOIC-8_5.23x5.23mm_P1.27mm
Changed lines of the file:
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@@
-    (pin "1")
-  )
-  (symbol (lib_id "Device:C_Small") (at 120.65 67.31 180) (unit 1)
-    (in_bom yes) (on_board yes)
-    (property "Reference" "C6" (id 0) (at 118.11 66.04 0)
-      (effects (font (size 1.27 1.27)) (justify left))
-    )
-    (property "Value" "100nF" (id 1) (at 118.11 68.58 0)
-      (effects (font (size 1.27 1.27)) (justify left))
-    )
-    (property "Footprint" "Capacitor_SMD:C_0402_1005Metric" (id 2) (at 120.65 67.31 0)
-      (effects (font (size 1.27 1.27)) hide)
-    )
-    (property "Datasheet" "~" (id 3) (at 120.65 67.31 0)
-      (effects (font (size 1.27 1.27)) hide)
-    )
-    (pin "1")
-    (pin "2")
-  )
-  (symbol (lib_id "Connector_Generic:Conn_01x01") (at 110.49 186.69 180) (unit 1)
-    (in_bom yes) (on_board yes)
-    (property "Reference" "J6" (id 0) (at 93.98 186.69 0))
-    (property "Value" "Conn_01x01" (id 1) (at 102.87 186.69 0))
-    (property "Footprint" "Connector_PinHeader_2.54mm:PinHeader_1x01_P2.54mm_Vertical" (id 2) (at 110.49 186.69 0)
-      (effects (font (size 1.27 1.27)) hide)
-    )
-    (property "Datasheet" "~" (id 3) (at 110.49 186.69 0)
-      (effects (font (size 1.27 1.27)) hide)
-    )
-    (pin "1")
-  )
-  (symbol (lib_id "power:PWR_FLAG") (at 185.42 33.02 0) (unit 1)
-    (in_bom yes) (on_board yes)
-    (property "Reference" "#FLG0101" (id 0) (at 185.42 31.115 0)
-      (effects (font (size 1.27 1.27)) hide)
-    )
-    (property "Value" "PWR_FLAG" (id 1) (at 182.88 29.21 0))
-    (property "Footprint" "" (id 2) (at 185.42 33.02 0)
-      (effects (font (size 1.27 1.27)) hide)
-    )
-    (property "Datasheet" "~" (id 3) (at 185.42 33.02 0)
-      (effects (font (size 1.27 1.27)) hide)
-    )
     (pin "1")
   )
@@
     (property "Reference" "U1" (id 0) (at 54.61 96.52 0))
     (property "Value" "W25Q128JVSIQTR" (id 1) (at 54.61 99.06 0))
-    (property "Footprint" "easyeda2kicad:SOIC-8_L5.3-W5.3-P1.27-LS8.0-BL" (id 2) (at 54.61 119.38 0)
+    (property "Footprint" "Package_SO:SOIC-8_5.23x5.23mm_P1.27mm" (id 2) (at 54.61 119.38 0)
       (effects (font (size 1.27 1.27)) hide)
     )
@@
     (pin "7")
     (pin "8")
+  )
+  (symbol (lib_id "Device:C_Small") (at 120.65 67.31 180) (unit 1)
+    (in_bom yes) (on_board yes)
+    (property "Reference" "C6" (id 0) (at 118.11 66.04 0)
+      (effects (font (size 1.27 1.27)) (justify left))
+    )
+    (property "Value" "100nF" (id 1) (at 118.11 68.58 0)
+      (effects (font (size 1.27 1.27)) (justify left))
+    )
+    (property "Footprint" "Capacitor_SMD:C_0402_1005Metric" (id 2) (at 120.65 67.31 0)
+      (effects (font (size 1.27 1.27)) hide)
+    )
+    (property "Datasheet" "~" (id 3) (at 120.65 67.31 0)
+      (effects (font (size 1.27 1.27)) hide)
+    )
+    (pin "1")
+    (pin "2")
+  )
+  (symbol (lib_id "Connector_Generic:Conn_01x01") (at 110.49 186.69 180) (unit 1)
+    (in_bom yes) (on_board yes)
+    (property "Reference" "J6" (id 0) (at 93.98 186.69 0))
+    (property "Value" "Conn_01x01" (id 1) (at 102.87 186.69 0))
+    (property "Footprint" "Connector_PinHeader_2.54mm:PinHeader_1x01_P2.54mm_Vertical" (id 2) (at 110.49 186.69 0)
+      (effects (font (size 1.27 1.27)) hide)
+    )
+    (property "Datasheet" "~" (id 3) (at 110.49 186.69 0)
+      (effects (font (size 1.27 1.27)) hide)
+    )
+    (pin "1")
+  )
+  (symbol (lib_id "power:PWR_FLAG") (at 185.42 33.02 0) (unit 1)
+    (in_bom yes) (on_board yes)
+    (property "Reference" "#FLG0101" (id 0) (at 185.42 31.115 0)
+      (effects (font (size 1.27 1.27)) hide)
+    )
+    (property "Value" "PWR_FLAG" (id 1) (at 182.88 29.21 0))
+    (property "Footprint" "" (id 2) (at 185.42 33.02 0)
+      (effects (font (size 1.27 1.27)) hide)
+    )
+    (property "Datasheet" "~" (id 3) (at 185.42 33.02 0)
+      (effects (font (size 1.27 1.27)) hide)
+    )
+    (pin "1")
   )
   (symbol (lib_id "power:GND") (at 157.48 36.83 0) (unit 1)
@@
   (symbol (lib_id "power:GND") (at 266.7 27.94 270) (unit 1)
     (in_bom yes) (on_board yes)
-    (property "Reference" "#PWR?" (id 0) (at 260.35 27.94 0)
+    (property "Reference" "#PWR0107" (id 0) (at 260.35 27.94 0)
       (effects (font (size 1.27 1.27)) hide)
     )
@@
     )
     (path "/fb79d012-1007-418b-b24e-637df639e8d0"
-      (reference "#PWR?") (unit 1) (value "GND") (footprint "")
+      (reference "#PWR0107") (unit 1) (value "GND") (footprint "")
     )
     (path "/80e37a29-2645-40c2-ad1a-3b8bdd51b77d/f56621e1-0429-4070-aa37-c7f1ca7e72ef"
@@
       (reference "R59") (unit 1) (value "470") (footprint "Resistor_SMD:R_0402_1005Metric")
     )
-    (path "/b5ef86b8-cc54-4119-ae66-7e751e9d7d90"
-      (reference "U1") (unit 1) (value "W25Q128JVSIQTR") (footprint "easyeda2kicad:SOIC-8_L5.3-W5.3-P1.27-LS8.0-BL")
+    (path "/b082fdb9-d1c4-4d81-8f42-8d2930dcd212"
+      (reference "U1") (unit 1) (value "W25Q128JVSIQTR") (footprint "Package_SO:SOIC-8_5.23x5.23mm_P1.27mm")
     )
     (path "/7b099bbc-3161-499b-9860-1aba9e193be0"
