File: Hardware/KiCad/projects/rp2040_v0/rp2040_v0/LEDs_and_buzzer.kicad_sch (KiCad schematic)
At the start: 9 parts, among them Q1 2N7002, Q3 2N7002

Commit message: Change LEDs to be kicad versions using kicad footprints for consistancy.
Parts:
- removed LED2: KT-0603R, easyeda2kicad:LED0603-R-RD, symbol easyeda2kicad_flight_computer:KT-0603R
- added D5: LED-KT-0603R, LED_SMD:LED_0603_1608Metric, symbol Device:LED
- D3: footprint easyeda2kicad:LED0603-R-RD -> LED_SMD:LED_0603_1608Metric
Connections:
- net at Q1.3 (D): now also D5.1 (K)
- net at R33.1: now also D5.2 (A)
Changed lines of the file:
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@@
     (stroke (width 0) (type default) (color 0 0 0 0))
   )
-  (wire (pts (xy 100.33 48.26) (xy 100.33 50.8))
+  (wire (pts (xy 100.33 48.26) (xy 100.33 52.07))
     (stroke (width 0) (type default) (color 0 0 0 0))
   )
@@
     (stroke (width 0) (type default) (color 0 0 0 0))
   )
-  (wire (pts (xy 100.33 60.96) (xy 100.33 64.77))
+  (wire (pts (xy 100.33 59.69) (xy 100.33 64.77))
     (stroke (width 0) (type default) (color 0 0 0 0))
   )
@@
       (effects (font (size 1.27 1.27)) (justify right))
     )
-    (property "Footprint" "easyeda2kicad:LED0603-R-RD" (id 2) (at 196.85 55.88 0)
+    (property "Footprint" "LED_SMD:LED_0603_1608Metric" (id 2) (at 196.85 55.88 0)
       (effects (font (size 1.27 1.27)) hide)
     )
     (property "Datasheet" "~" (id 3) (at 196.85 55.88 0)
+      (effects (font (size 1.27 1.27)) hide)
+    )
+    (pin "1")
+    (pin "2")
+  )
+  (symbol (lib_id "Device:LED") (at 100.33 55.88 90) (unit 1)
+    (in_bom yes) (on_board yes) (fields_autoplaced)
+    (property "Reference" "D5" (id 0) (at 104.14 56.1974 90)
+      (effects (font (size 1.27 1.27)) (justify right))
+    )
+    (property "Value" "LED-KT-0603R" (id 1) (at 104.14 58.7374 90)
+      (effects (font (size 1.27 1.27)) (justify right))
+    )
+    (property "Footprint" "LED_SMD:LED_0603_1608Metric" (id 2) (at 100.33 55.88 0)
+      (effects (font (size 1.27 1.27)) hide)
+    )
+    (property "Datasheet" "~" (id 3) (at 100.33 55.88 0)
       (effects (font (size 1.27 1.27)) hide)
     )
@@
     (pin "1")
   )
-  (symbol (lib_id "easyeda2kicad_flight_computer:KT-0603R") (at 101.6 55.88 90) (unit 1)
-    (in_bom yes) (on_board yes) (fields_autoplaced)
-    (property "Reference" "LED2" (id 0) (at 105.41 55.8799 90)
-      (effects (font (size 1.27 1.27)) (justify right))
-    )
-    (property "Value" "KT-0603R" (id 1) (at 105.41 58.4199 90)
-      (effects (font (size 1.27 1.27)) (justify right))
-    )
-    (property "Footprint" "easyeda2kicad:LED0603-R-RD" (id 2) (at 107.95 55.88 0)
-      (effects (font (size 1.27 1.27)) hide)
-    )
-    (property "Datasheet" "https://lcsc.com/product-detail/Light-Emitting-Diodes-LED_Red-LED-0603_C2286.html" (id 3) (at 110.49 55.88 0)
-      (effects (font (size 1.27 1.27)) hide)
-    )
-    (property "LCSC Part" "C2286" (id 4) (at 113.03 55.88 0)
-      (effects (font (size 1.27 1.27)) hide)
-    )
-    (property "JLC Part" "Basic Part" (id 5) (at 115.57 55.88 0)
-      (effects (font (size 1.27 1.27)) hide)
-    )
-    (pin "1")
-    (pin "2")
-  )
   (symbol (lib_id "Device:R_Small") (at 196.85 45.72 180) (unit 1)
