File: Hardware/KiCad/projects/rp2040_v0/rp2040_v0/LEDs_and_buzzer.kicad_sch (KiCad schematic)
At the start: 9 parts, among them Q1 2N7002, Q3 2N7002

Commit message: Rev 0 ready to ship! Had to move IMU so board got sloppy. IMU should be in the middle of the board. Glad I caught that.
Parts:
- BZ1: JLC Part (none) -> Extended Part; LCSC Part (none) -> C161819
- D3: JLC Part (none) -> Basic Part; LCSC Part (none) -> C72043
- D5: JLC Part (none) -> Basic Part; LCSC Part (none) -> C2286
- Q1, Q3: JLC Part (none) -> Basic Part; LCSC Part (none) -> C8545
- R10, R32: JLC Part (none) -> Basic Part; LCSC Part (none) -> C25117
- R11: JLC Part (none) -> Basic Part; LCSC Part (none) -> C25076
- R33: JLC Part (none) -> Basic Part; LCSC Part (none) -> C25087
Changed lines of the file:
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@@
       (effects (font (size 1.27 1.27)) (justify left) hide)
+    )
+    (property "LCSC Part" "C8545" (id 4) (at 97.79 69.85 0)
+      (effects (font (size 1.27 1.27)) hide)
+    )
+    (property "JLC Part" "Basic Part" (id 5) (at 97.79 69.85 0)
+      (effects (font (size 1.27 1.27)) hide)
     )
     (pin "1")
@@
       (effects (font (size 1.27 1.27)) hide)
     )
+    (property "LCSC Part" "C25117" (id 4) (at 82.55 69.85 0)
+      (effects (font (size 1.27 1.27)) hide)
+    )
+    (property "JLC Part" "Basic Part" (id 5) (at 82.55 69.85 0)
+      (effects (font (size 1.27 1.27)) hide)
+    )
     (pin "1")
     (pin "2")
@@
       (effects (font (size 1.27 1.27)) hide)
     )
+    (property "LCSC Part" "C72043" (id 4) (at 196.85 55.88 0)
+      (effects (font (size 1.27 1.27)) hide)
+    )
+    (property "JLC Part" "Basic Part" (id 5) (at 196.85 55.88 0)
+      (effects (font (size 1.27 1.27)) hide)
+    )
     (pin "1")
     (pin "2")
@@
     )
     (property "Datasheet" "~" (id 3) (at 100.33 55.88 0)
+      (effects (font (size 1.27 1.27)) hide)
+    )
+    (property "LCSC Part" "C2286" (id 4) (at 100.33 55.88 0)
+      (effects (font (size 1.27 1.27)) hide)
+    )
+    (property "JLC Part" "Basic Part" (id 5) (at 100.33 55.88 0)
       (effects (font (size 1.27 1.27)) hide)
     )
@@
       (effects (font (size 1.27 1.27)) hide)
     )
+    (property "LCSC Part" "C25076" (id 4) (at 196.85 45.72 0)
+      (effects (font (size 1.27 1.27)) hide)
+    )
+    (property "JLC Part" "Basic Part" (id 5) (at 196.85 45.72 0)
+      (effects (font (size 1.27 1.27)) hide)
+    )
     (pin "1")
     (pin "2")
@@
     (property "Datasheet" "https://www.onsemi.com/pub/Collateral/NDS7002A-D.PDF" (id 3) (at 194.31 69.85 0)
       (effects (font (size 1.27 1.27)) (justify left) hide)
+    )
+    (property "LCSC Part" "C8545" (id 4) (at 194.31 69.85 0)
+      (effects (font (size 1.27 1.27)) hide)
+    )
+    (property "JLC Part" "Basic Part" (id 5) (at 194.31 69.85 0)
+      (effects (font (size 1.27 1.27)) hide)
     )
     (pin "1")
@@
       (effects (font (size 1.27 1.27)) hide)
     )
+    (property "LCSC Part" "C25117" (id 4) (at 179.07 69.85 0)
+      (effects (font (size 1.27 1.27)) hide)
+    )
+    (property "JLC Part" "Basic Part" (id 5) (at 179.07 69.85 0)
+      (effects (font (size 1.27 1.27)) hide)
+    )
     (pin "1")
     (pin "2")
@@
       (effects (font (size 1.27 1.27)) hide)
     )
+    (property "LCSC Part" "C161819" (id 4) (at 68.58 152.4 0)
+      (effects (font (size 1.27 1.27)) hide)
+    )
+    (property "JLC Part" "Extended Part" (id 5) (at 68.58 152.4 0)
+      (effects (font (size 1.27 1.27)) hide)
+    )
     (pin "1")
     (pin "2")
@@
       (effects (font (size 1.27 1.27)) hide)
     )
+    (property "LCSC Part" "C25087" (id 4) (at 100.33 45.72 0)
+      (effects (font (size 1.27 1.27)) hide)
+    )
+    (property "JLC Part" "Basic Part" (id 5) (at 100.33 45.72 0)
+      (effects (font (size 1.27 1.27)) hide)
+    )

Commit message: Some minor changes with footprint. Sent to JLCPCB. Official Rev 0!
Parts:
- BZ1: LCSC (none) -> C161819
- D3: LCSC (none) -> C72043
- D5: LCSC (none) -> C2286
- Q1, Q3: LCSC (none) -> C8545
- R10, R32: LCSC (none) -> C25117
- R11: LCSC (none) -> C25076
- R33: LCSC (none) -> C25087
Changed lines of the file:
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@@
+      (effects (font (size 1.27 1.27)) hide)
+    )
+    (property "LCSC" "C8545" (id 6) (at 97.79 69.85 0)
       (effects (font (size 1.27 1.27)) hide)
     )
@@
       (effects (font (size 1.27 1.27)) hide)
     )
+    (property "LCSC" "C25117" (id 6) (at 82.55 69.85 0)
+      (effects (font (size 1.27 1.27)) hide)
+    )
     (pin "1")
     (pin "2")
@@
       (effects (font (size 1.27 1.27)) hide)
     )
+    (property "LCSC" "C72043" (id 6) (at 196.85 55.88 0)
+      (effects (font (size 1.27 1.27)) hide)
+    )
     (pin "1")
     (pin "2")
@@
     )
     (property "JLC Part" "Basic Part" (id 5) (at 100.33 55.88 0)
+      (effects (font (size 1.27 1.27)) hide)
+    )
+    (property "LCSC" "C2286" (id 6) (at 100.33 55.88 0)
       (effects (font (size 1.27 1.27)) hide)
     )
@@
       (effects (font (size 1.27 1.27)) hide)
     )
+    (property "LCSC" "C25076" (id 6) (at 196.85 45.72 0)
+      (effects (font (size 1.27 1.27)) hide)
+    )
     (pin "1")
     (pin "2")
@@
     )
     (property "JLC Part" "Basic Part" (id 5) (at 194.31 69.85 0)
+      (effects (font (size 1.27 1.27)) hide)
+    )
+    (property "LCSC" "C8545" (id 6) (at 194.31 69.85 0)
       (effects (font (size 1.27 1.27)) hide)
     )
@@
       (effects (font (size 1.27 1.27)) hide)
     )
+    (property "LCSC" "C25117" (id 6) (at 179.07 69.85 0)
+      (effects (font (size 1.27 1.27)) hide)
+    )
     (pin "1")
     (pin "2")
@@
       (effects (font (size 1.27 1.27)) hide)
     )
+    (property "LCSC" "C161819" (id 6) (at 68.58 152.4 0)
+      (effects (font (size 1.27 1.27)) hide)
+    )
     (pin "1")
     (pin "2")
@@
       (effects (font (size 1.27 1.27)) hide)
     )
+    (property "LCSC" "C25087" (id 6) (at 100.33 45.72 0)
+      (effects (font (size 1.27 1.27)) hide)
+    )
