File: Hardware/KiCad/projects/rp2040_v0/rp2040_v0/IMU.kicad_sch (KiCad schematic)
At the start: 13 parts, among them J13 Conn_02x09_Counter_Clockwise, U5 BMI088

Commit message: Change LEDs to be kicad versions using kicad footprints for consistancy.
Parts:
- removed J13: Conn_02x09_Counter_Clockwise, Connector_PinHeader_2.54mm:PinHeader_2x09_P2.54mm_Vertical, symbol Connector_Generic:Conn_02x09_Counter_Clockwise
- added J13: Conn_02x09_Odd_Even, Connector_PinHeader_2.54mm:PinHeader_2x09_P2.54mm_Vertical, symbol Connector_Generic:Conn_02x09_Odd_Even
Connections:
- net +3.3V: now also J13.12 (Pin_12)
- net ACCEL_INT: now also J13.4 (Pin_4)
- net GYRO_INT: now also J13.10 (Pin_10)
- net SPI0_CSn__BMI088_CS_ACCEL: now also J13.8 (Pin_8)
- net SPI0_CSn__BMI088_CS_GYRO: now also J13.2 (Pin_2)
- net SPI0_RX__BMI088_MISO: now also J13.14 (Pin_14), J13.6 (Pin_6)
- net SPI0_SCK__BMI088_SCLK: now also J13.18 (Pin_18)
- net SPI0_TX__BMI088_MOSI: now also J13.16 (Pin_16)
- net at R18.1, U5.10 (SDO2): now also J13.13 (Pin_13)
- net at R12.1, U5.16 (INT1): now also J13.3 (Pin_3)
- net at C20.1, C21.1, R17.1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: now also J13.11 (Pin_11)
- net at R16.1, U5.12 (INT3): now also J13.9 (Pin_9)
- net at R14.1, U5.14 (CSB1): now also J13.7 (Pin_7)
- net at R13.1, U5.15 (SDO1): now also J13.5 (Pin_5)
- net at R9.1, U5.5 (CSB2): now also J13.1 (Pin_1)
- net at R20.1, U5.8 (SCL/SCK): now also J13.17 (Pin_17)
- net at R19.1, U5.9 (SDA/SDI): now also J13.15 (Pin_15)
Changed lines of the file:
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@@
     (pin "2")
+  )
+  (symbol (lib_id "Connector_Generic:Conn_02x09_Odd_Even") (at 223.52 91.44 0) (unit 1)
+    (in_bom yes) (on_board yes) (fields_autoplaced)
+    (property "Reference" "J13" (id 0) (at 224.79 74.93 0))
+    (property "Value" "Conn_02x09_Odd_Even" (id 1) (at 224.79 77.47 0))
+    (property "Footprint" "Connector_PinHeader_2.54mm:PinHeader_2x09_P2.54mm_Vertical" (id 2) (at 223.52 91.44 0)
+      (effects (font (size 1.27 1.27)) hide)
+    )
+    (property "Datasheet" "~" (id 3) (at 223.52 91.44 0)
+      (effects (font (size 1.27 1.27)) hide)
+    )
+    (pin "1")
+    (pin "10")
+    (pin "11")
+    (pin "12")
+    (pin "13")
+    (pin "14")
+    (pin "15")
+    (pin "16")
+    (pin "17")
+    (pin "18")
+    (pin "2")
+    (pin "3")
+    (pin "4")
+    (pin "5")
+    (pin "6")
+    (pin "7")
+    (pin "8")
+    (pin "9")
   )
   (symbol (lib_id "power:GND") (at 87.63 100.33 0) (unit 1)
@@
     (pin "2")
   )
-  (symbol (lib_id "Connector_Generic:Conn_02x09_Counter_Clockwise") (at 223.52 91.44 0) (unit 1)
-    (in_bom yes) (on_board yes) (fields_autoplaced)
-    (property "Reference" "J13" (id 0) (at 224.79 74.93 0))
-    (property "Value" "Conn_02x09_Counter_Clockwise" (id 1) (at 224.79 77.47 0))
-    (property "Footprint" "Connector_PinHeader_2.54mm:PinHeader_2x09_P2.54mm_Vertical" (id 2) (at 223.52 91.44 0)
-      (effects (font (size 1.27 1.27)) hide)
-    )
-    (property "Datasheet" "~" (id 3) (at 223.52 91.44 0)
-      (effects (font (size 1.27 1.27)) hide)
-    )
-    (pin "1")
-    (pin "10")
-    (pin "11")
-    (pin "12")
-    (pin "13")
-    (pin "14")
-    (pin "15")
-    (pin "16")
-    (pin "17")
-    (pin "18")
-    (pin "2")
-    (pin "3")
-    (pin "4")
-    (pin "5")
-    (pin "6")
-    (pin "7")
-    (pin "8")
-    (pin "9")
-  )
   (symbol (lib_id "power:+3.3V") (at 240.03 138.43 270) (mirror x) (unit 1)

Commit message: Change some header pin pinouts to make routing easier.
Connections:
- net +3.3V: now also J13.8 (Pin_8), R14.2; no longer J13.12 (Pin_12), R17.2
- net ACCEL_INT: now also J13.16 (Pin_16), R19.2; no longer J13.4 (Pin_4), R12.2
- net SPI0_CSn__BMI088_CS_ACCEL: now also J13.12 (Pin_12), R17.2; no longer J13.8 (Pin_8), R14.2
- net SPI0_CSn__BMI088_CS_GYRO: now also J13.18 (Pin_18), R20.2; no longer J13.2 (Pin_2), R9.2
- net SPI0_RX__BMI088_MISO: no longer J13.6 (Pin_6)
- net SPI0_SCK__BMI088_SCLK: now also J13.2 (Pin_2), R9.2; no longer J13.18 (Pin_18), R20.2
- net SPI0_TX__BMI088_MOSI: now also J13.4 (Pin_4), R12.2; no longer J13.16 (Pin_16), R19.2
- net at J13.13 (Pin_13), R18.1: now also U5.15 (SDO1); no longer U5.10 (SDO2)
- net at J13.3 (Pin_3), R12.1: now also U5.9 (SDA/SDI); no longer U5.16 (INT1)
- net at C20.1, C21.1, U5.11 (VDDIO)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: now also J13.7 (Pin_7), R14.1; no longer J13.11 (Pin_11), R17.1
- net at J13.5 (Pin_5), R13.1: now also U5.10 (SDO2); no longer U5.15 (SDO1)
- net at J13.1 (Pin_1), R9.1: now also U5.8 (SCL/SCK); no longer U5.5 (CSB2)
- net at J13.17 (Pin_17), R20.1: now also U5.5 (CSB2); no longer U5.8 (SCL/SCK)
- net at J13.15 (Pin_15), R19.1: now also U5.16 (INT1); no longer U5.9 (SDA/SDI)
- new net: J13.11 (Pin_11), R17.1, U5.14 (CSB1)
Other:
- moved on the sheet: R12, R13, R14, R17, R18, R19, R20, R9

Commit message: Whoops - reconnect IMU pin that accidently got removed.
Connections:
- net SPI0_RX__BMI088_MISO: now also J13.6 (Pin_6)
Changed lines of the file:
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@@
     (stroke (width 0) (type default) (color 0 0 0 0))
   )
-  (wire (pts (xy 233.68 96.52) (xy 236.22 96.52))
+  (wire (pts (xy 231.14 96.52) (xy 236.22 96.52))
     (stroke (width 0) (type default) (color 0 0 0 0))
   )
