File: Hardware/KiCad/projects/rp2040_v0/rp2040_v0/Barometer.kicad_sch (KiCad schematic)
At the start: 10 parts, among them J14 Conn_02x06_Odd_Even, U6 BMP280

Commit message: Rev 0 ready to ship! Had to move IMU so board got sloppy. IMU should be in the middle of the board. Glad I caught that.
Parts:
- C22, C23: JLC Part (none) -> Basic Part; LCSC Part (none) -> C307331
- R21, R22, R23, R24, R25, R26: JLC Part (none) -> Basic Part; LCSC Part (none) -> C17168
- U6: JLC Part (none) -> Extended Part; LCSC Part (none) -> C83291
Changed lines of the file:
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@@
+      (effects (font (size 1.27 1.27)) hide)
+    )
+    (property "LCSC Part" "C17168" (id 4) (at 125.73 104.14 0)
+      (effects (font (size 1.27 1.27)) hide)
+    )
+    (property "JLC Part" "Basic Part" (id 5) (at 125.73 104.14 0)
       (effects (font (size 1.27 1.27)) hide)
     )
@@
     )
     (property "Datasheet" "~" (id 3) (at 125.73 101.6 0)
+      (effects (font (size 1.27 1.27)) hide)
+    )
+    (property "LCSC Part" "C17168" (id 4) (at 125.73 101.6 0)
+      (effects (font (size 1.27 1.27)) hide)
+    )
+    (property "JLC Part" "Basic Part" (id 5) (at 125.73 101.6 0)
       (effects (font (size 1.27 1.27)) hide)
     )
@@
     )
     (property "Datasheet" "https://ae-bst.resource.bosch.com/media/_tech/media/datasheets/BST-BMP280-DS001.pdf" (id 3) (at 172.72 83.82 0)
+      (effects (font (size 1.27 1.27)) hide)
+    )
+    (property "LCSC Part" "C83291" (id 4) (at 172.72 83.82 0)
+      (effects (font (size 1.27 1.27)) hide)
+    )
+    (property "JLC Part" "Extended Part" (id 5) (at 172.72 83.82 0)
       (effects (font (size 1.27 1.27)) hide)
     )
@@
       (effects (font (size 1.27 1.27)) hide)
     )
+    (property "LCSC Part" "C17168" (id 4) (at 125.73 106.68 0)
+      (effects (font (size 1.27 1.27)) hide)
+    )
+    (property "JLC Part" "Basic Part" (id 5) (at 125.73 106.68 0)
+      (effects (font (size 1.27 1.27)) hide)
+    )
     (pin "1")
     (pin "2")
@@
     )
     (property "Datasheet" "~" (id 3) (at 125.73 109.22 0)
+      (effects (font (size 1.27 1.27)) hide)
+    )
+    (property "LCSC Part" "C17168" (id 4) (at 125.73 109.22 0)
+      (effects (font (size 1.27 1.27)) hide)
+    )
+    (property "JLC Part" "Basic Part" (id 5) (at 125.73 109.22 0)
       (effects (font (size 1.27 1.27)) hide)
     )
@@
       (effects (font (size 1.27 1.27)) hide)
     )
+    (property "LCSC Part" "C307331" (id 4) (at 177.8 68.58 0)
+      (effects (font (size 1.27 1.27)) hide)
+    )
+    (property "JLC Part" "Basic Part" (id 5) (at 177.8 68.58 0)
+      (effects (font (size 1.27 1.27)) hide)
+    )
     (pin "1")
     (pin "2")
@@
       (effects (font (size 1.27 1.27)) hide)
     )
+    (property "LCSC Part" "C17168" (id 4) (at 125.73 111.76 0)
+      (effects (font (size 1.27 1.27)) hide)
+    )
+    (property "JLC Part" "Basic Part" (id 5) (at 125.73 111.76 0)
+      (effects (font (size 1.27 1.27)) hide)
+    )
     (pin "1")
     (pin "2")
@@
       (effects (font (size 1.27 1.27)) hide)
     )
+    (property "LCSC Part" "C307331" (id 4) (at 168.91 68.58 0)
+      (effects (font (size 1.27 1.27)) hide)
+    )
+    (property "JLC Part" "Basic Part" (id 5) (at 168.91 68.58 0)
+      (effects (font (size 1.27 1.27)) hide)
+    )
     (pin "1")
     (pin "2")
@@
       (effects (font (size 1.27 1.27)) hide)
     )
+    (property "LCSC Part" "C17168" (id 4) (at 125.73 114.3 0)
+      (effects (font (size 1.27 1.27)) hide)
+    )
+    (property "JLC Part" "Basic Part" (id 5) (at 125.73 114.3 0)
+      (effects (font (size 1.27 1.27)) hide)
+    )

Commit message: Some minor changes with footprint. Sent to JLCPCB. Official Rev 0!
Parts:
- C22, C23: LCSC (none) -> C307331
- R21, R22, R23, R24, R25, R26: LCSC (none) -> C17168
- U6: LCSC (none) -> C83291
Changed lines of the file:
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@@
+      (effects (font (size 1.27 1.27)) hide)
+    )
+    (property "LCSC" "C17168" (id 6) (at 125.73 104.14 0)
       (effects (font (size 1.27 1.27)) hide)
     )
@@
     )
     (property "JLC Part" "Basic Part" (id 5) (at 125.73 101.6 0)
+      (effects (font (size 1.27 1.27)) hide)
+    )
+    (property "LCSC" "C17168" (id 6) (at 125.73 101.6 0)
       (effects (font (size 1.27 1.27)) hide)
     )
@@
     )
     (property "JLC Part" "Extended Part" (id 5) (at 172.72 83.82 0)
+      (effects (font (size 1.27 1.27)) hide)
+    )
+    (property "LCSC" "C83291" (id 6) (at 172.72 83.82 0)
       (effects (font (size 1.27 1.27)) hide)
     )
@@
       (effects (font (size 1.27 1.27)) hide)
     )
+    (property "LCSC" "C17168" (id 6) (at 125.73 106.68 0)
+      (effects (font (size 1.27 1.27)) hide)
+    )
     (pin "1")
     (pin "2")
@@
     )
     (property "JLC Part" "Basic Part" (id 5) (at 125.73 109.22 0)
+      (effects (font (size 1.27 1.27)) hide)
+    )
+    (property "LCSC" "C17168" (id 6) (at 125.73 109.22 0)
       (effects (font (size 1.27 1.27)) hide)
     )
@@
       (effects (font (size 1.27 1.27)) hide)
     )
+    (property "LCSC" "C307331" (id 6) (at 177.8 68.58 0)
+      (effects (font (size 1.27 1.27)) hide)
+    )
     (pin "1")
     (pin "2")
@@
       (effects (font (size 1.27 1.27)) hide)
     )
+    (property "LCSC" "C17168" (id 6) (at 125.73 111.76 0)
+      (effects (font (size 1.27 1.27)) hide)
+    )
     (pin "1")
     (pin "2")
@@
       (effects (font (size 1.27 1.27)) hide)
     )
+    (property "LCSC" "C307331" (id 6) (at 168.91 68.58 0)
+      (effects (font (size 1.27 1.27)) hide)
+    )
     (pin "1")
     (pin "2")
@@
       (effects (font (size 1.27 1.27)) hide)
     )
+    (property "LCSC" "C17168" (id 6) (at 125.73 114.3 0)
+      (effects (font (size 1.27 1.27)) hide)
+    )
