File: Hardware/KiCad/projects/rp2040_v0/rp2040_v0/Servos.kicad_sch (KiCad schematic)
At the start: 11 parts, among them J17 Conn_01x03, J18 Conn_01x03, J19 Conn_01x03, J20 Conn_01x03, J21 Conn_01x03, U7 AMS1117-5.0, U8 AMS1117-5.0

Commit message: Rev 0 ready to ship! Had to move IMU so board got sloppy. IMU should be in the middle of the board. Glad I caught that.
Parts:
- C24, C25, C27, C28: JLC Part (none) -> Basic Part; LCSC Part (none) -> C15850
- U7, U8: JLC Part (none) -> Basic Part; LCSC Part (none) -> C6187
Changed lines of the file:
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@@
+      (effects (font (size 1.27 1.27)) hide)
+    )
+    (property "LCSC Part" "C6187" (id 4) (at 46.99 121.92 0)
+      (effects (font (size 1.27 1.27)) hide)
+    )
+    (property "JLC Part" "Basic Part" (id 5) (at 46.99 121.92 0)
       (effects (font (size 1.27 1.27)) hide)
     )
@@
     )
     (property "Datasheet" "http://www.advanced-monolithic.com/pdf/ds1117.pdf" (id 3) (at 49.53 149.86 0)
+      (effects (font (size 1.27 1.27)) hide)
+    )
+    (property "LCSC Part" "C6187" (id 4) (at 46.99 143.51 0)
+      (effects (font (size 1.27 1.27)) hide)
+    )
+    (property "JLC Part" "Basic Part" (id 5) (at 46.99 143.51 0)
       (effects (font (size 1.27 1.27)) hide)
     )
@@
     )
     (property "Datasheet" "~" (id 3) (at 38.1 146.05 0)
+      (effects (font (size 1.27 1.27)) hide)
+    )
+    (property "LCSC Part" "C15850" (id 4) (at 38.1 146.05 0)
+      (effects (font (size 1.27 1.27)) hide)
+    )
+    (property "JLC Part" "Basic Part" (id 5) (at 38.1 146.05 0)
       (effects (font (size 1.27 1.27)) hide)
     )
@@
       (effects (font (size 1.27 1.27)) hide)
     )
+    (property "LCSC Part" "C15850" (id 4) (at 55.88 146.05 0)
+      (effects (font (size 1.27 1.27)) hide)
+    )
+    (property "JLC Part" "Basic Part" (id 5) (at 55.88 146.05 0)
+      (effects (font (size 1.27 1.27)) hide)
+    )
     (pin "1")
     (pin "2")
@@
       (effects (font (size 1.27 1.27)) hide)
     )
+    (property "LCSC Part" "C15850" (id 4) (at 38.1 124.46 0)
+      (effects (font (size 1.27 1.27)) hide)
+    )
+    (property "JLC Part" "Basic Part" (id 5) (at 38.1 124.46 0)
+      (effects (font (size 1.27 1.27)) hide)
+    )
     (pin "1")
     (pin "2")
@@
       (effects (font (size 1.27 1.27)) hide)
     )
+    (property "LCSC Part" "C15850" (id 4) (at 55.88 124.46 0)
+      (effects (font (size 1.27 1.27)) hide)
+    )
+    (property "JLC Part" "Basic Part" (id 5) (at 55.88 124.46 0)
+      (effects (font (size 1.27 1.27)) hide)
+    )

Commit message: Some minor changes with footprint. Sent to JLCPCB. Official Rev 0!
Parts:
- C24, C25, C27, C28: LCSC (none) -> C15850
- U7, U8: LCSC (none) -> C6187
Changed lines of the file:
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@@
+      (effects (font (size 1.27 1.27)) hide)
+    )
+    (property "LCSC" "C6187" (id 6) (at 46.99 121.92 0)
       (effects (font (size 1.27 1.27)) hide)
     )
@@
     )
     (property "JLC Part" "Basic Part" (id 5) (at 46.99 143.51 0)
+      (effects (font (size 1.27 1.27)) hide)
+    )
+    (property "LCSC" "C6187" (id 6) (at 46.99 143.51 0)
       (effects (font (size 1.27 1.27)) hide)
     )
@@
     )
     (property "JLC Part" "Basic Part" (id 5) (at 38.1 146.05 0)
+      (effects (font (size 1.27 1.27)) hide)
+    )
+    (property "LCSC" "C15850" (id 6) (at 38.1 146.05 0)
       (effects (font (size 1.27 1.27)) hide)
     )
@@
       (effects (font (size 1.27 1.27)) hide)
     )
+    (property "LCSC" "C15850" (id 6) (at 55.88 146.05 0)
+      (effects (font (size 1.27 1.27)) hide)
+    )
     (pin "1")
     (pin "2")
@@
       (effects (font (size 1.27 1.27)) hide)
     )
+    (property "LCSC" "C15850" (id 6) (at 38.1 124.46 0)
+      (effects (font (size 1.27 1.27)) hide)
+    )
     (pin "1")
     (pin "2")
@@
       (effects (font (size 1.27 1.27)) hide)
     )
+    (property "LCSC" "C15850" (id 6) (at 55.88 124.46 0)
+      (effects (font (size 1.27 1.27)) hide)
+    )
